File: 24S_Counter.kicad_sch (KiCad schematic)
At the start: 32 parts, among them J1 +5V, J2 EXT_CLK, SW1 EN, SW2 RST, U1 74LS192, U2 74LS192, U3 74LS48, U4 74LS48, U5 SM420561N, U6 SM420561N

Commit message: Edited PCB Design
Parts:
- J1: footprint (none) -> my_footprints:Terminal_Block_5mm
- SW1: footprint (none) -> my_footprints:slide_switch_2.54mm
- SW2: footprint (none) -> my_footprints:tact_switch_5mm
- U1, U2: footprint (none) -> my_footprints:74LS192
- U3, U4: footprint (none) -> my_footprints:74LS48
Changed lines of the file:
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@@
 			)
 		)
-		(property "Footprint" ""
+		(property "Footprint" "my_footprints:slide_switch_2.54mm"
 			(at 187.96 83.82 0)
 			(effects
@@
 			)
 		)
-		(property "Footprint" ""
+		(property "Footprint" "my_footprints:74LS48"
 			(at 114.3 106.68 0)
 			(effects
@@
 			)
 		)
-		(property "Footprint" ""
+		(property "Footprint" "my_footprints:tact_switch_5mm"
 			(at 190.5 35.56 0)
 			(effects
@@
 			)
 		)
-		(property "Footprint" ""
+		(property "Footprint" "my_footprints:74LS192"
 			(at 83.82 48.26 0)
 			(effects
@@
 			)
 		)
-		(property "Footprint" ""
+		(property "Footprint" "my_footprints:74LS48"
 			(at 114.3 45.72 0)
 			(effects
@@
 			)
 		)
-		(property "Footprint" ""
+		(property "Footprint" "my_footprints:Terminal_Block_5mm"
 			(at 196.85 113.03 0)
 			(effects
@@
 			)
 		)
-		(property "Footprint" ""
+		(property "Footprint" "my_footprints:74LS192"
 			(at 83.82 109.22 0)
 			(effects
