File: 24S_Counter.kicad_pcb (KiCad board)
At the start: 2 copper layers, 0 parts

Commit message: Edited PCB Design
Parts:
- added H1: MountingHole, MountingHole:MountingHole_2.2mm_M2, F.Cu at (57.7, 152.0)
- added H2: MountingHole, MountingHole:MountingHole_2.2mm_M2, F.Cu at (57.7, 157.9)
- added H3: MountingHole, MountingHole:MountingHole_2.2mm_M2, F.Cu at (57.7, 163.9)
- added H4: MountingHole, MountingHole:MountingHole_2.2mm_M2, F.Cu at (57.7, 169.8)
- added J1: +5V, my_footprints:Terminal_Block_5mm, F.Cu at (99.2, 70.2)
- added J2: EXT_CLK, Connector_PinHeader_2.54mm:PinHeader_1x02_P2.54mm_Vertical, F.Cu at (96.6, 112.0)
- added R1: 100R, Resistor_SMD:R_1206_3216Metric_Pad1.30x1.75mm_HandSolder, F.Cu at (125.6, 82.0)
- added R10: 100R, Resistor_SMD:R_1206_3216Metric_Pad1.30x1.75mm_HandSolder, F.Cu at (161.0, 116.2)
- added R11: 100R, Resistor_SMD:R_1206_3216Metric_Pad1.30x1.75mm_HandSolder, F.Cu at (161.0, 120.1)
- added R12: 100R, Resistor_SMD:R_1206_3216Metric_Pad1.30x1.75mm_HandSolder, F.Cu at (161.0, 123.9)
- added R13: 100R, Resistor_SMD:R_1206_3216Metric_Pad1.30x1.75mm_HandSolder, F.Cu at (154.3, 74.9)
- added R14: 100R, Resistor_SMD:R_1206_3216Metric_Pad1.30x1.75mm_HandSolder, F.Cu at (148.1, 74.9)
- added R15: 1K, Resistor_SMD:R_1206_3216Metric_Pad1.30x1.75mm_HandSolder, F.Cu at (120.1, 120.9)
- added R16: 10K, Resistor_SMD:R_1206_3216Metric_Pad1.30x1.75mm_HandSolder, F.Cu at (120.1, 117.0)
- added R17: 1K, Resistor_SMD:R_1206_3216Metric_Pad1.30x1.75mm_HandSolder, F.Cu at (102.6, 116.3)
- added R18: 10K, Resistor_SMD:R_1206_3216Metric_Pad1.30x1.75mm_HandSolder, F.Cu at (102.6, 110.1)
- added R2: 100R, Resistor_SMD:R_1206_3216Metric_Pad1.30x1.75mm_HandSolder, F.Cu at (125.7, 86.1)
- added R3: 100R, Resistor_SMD:R_1206_3216Metric_Pad1.30x1.75mm_HandSolder, F.Cu at (125.7, 90.2)
- added R4: 100R, Resistor_SMD:R_1206_3216Metric_Pad1.30x1.75mm_HandSolder, F.Cu at (125.7, 94.3)
- added R5: 100R, Resistor_SMD:R_1206_3216Metric_Pad1.30x1.75mm_HandSolder, F.Cu at (125.7, 98.3)
- added R6: 100R, Resistor_SMD:R_1206_3216Metric_Pad1.30x1.75mm_HandSolder, F.Cu at (135.3, 74.9)
- added R7: 100R, Resistor_SMD:R_1206_3216Metric_Pad1.30x1.75mm_HandSolder, F.Cu at (125.6, 78.0)
- added R8: 100R, Resistor_SMD:R_1206_3216Metric_Pad1.30x1.75mm_HandSolder, F.Cu at (161.0, 107.9)
- added R9: 100R, Resistor_SMD:R_1206_3216Metric_Pad1.30x1.75mm_HandSolder, F.Cu at (161.0, 112.2)
- added SW1: EN, my_footprints:slide_switch_2.54mm, F.Cu at (109.3, 113.3)
- added SW2: RST, my_footprints:tact_switch_5mm, F.Cu at (119.8, 110.5)
- added U1: 74LS192, my_footprints:74LS192, F.Cu at (98.5, 89.5)
- added U2: 74LS192, my_footprints:74LS192, F.Cu at (134.1, 114.9)
- added U3: 74LS48, my_footprints:74LS48, F.Cu at (112.5, 89.4)
- added U4: 74LS48, my_footprints:74LS48, F.Cu at (148.3, 114.9)
- added U5: SM420561N, Display_7Segment:7SegmentLED_LTS6760_LTS6780, F.Cu at (134.4, 95.5)
- added U6: SM420561N, Display_7Segment:7SegmentLED_LTS6760_LTS6780, F.Cu at (150.2, 95.5)
Routing:
- net GND: track 0.00 -> 222.7 mm
- net /+5V: track 0.00 -> 165.2 mm, vias 0 -> 3
- net /Load: track 0.00 -> 69.7 mm, vias 0 -> 1
- net /B0: track 0.00 -> 68.5 mm
- net Net-(U6-E): track 0.00 -> 45.3 mm, vias 0 -> 1
- net Net-(U4-f): track 0.00 -> 42.9 mm
- net Net-(U1-QC): track 0.00 -> 40.6 mm
- net Net-(U2-QC): track 0.00 -> 39.4 mm
- net Net-(U4-g): track 0.00 -> 38.4 mm
- net Net-(U6-B): track 0.00 -> 34.7 mm, vias 0 -> 1
- net Net-(U1-QA): track 0.00 -> 33.9 mm
- net Net-(U1-QD): track 0.00 -> 32.3 mm, vias 0 -> 1
- net /CLK: track 0.00 -> 32.1 mm, vias 0 -> 1
- net Net-(U6-D): track 0.00 -> 30.7 mm, vias 0 -> 1
- net Net-(U6-A): track 0.00 -> 30.3 mm, vias 0 -> 1
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
Commit message: Updated PCB Design
Parts:
- added G***: LOGO, Special_Footprints:BoyKisser11x11mm, F.Cu at (120.4, 125.0)
- added G***: LOGO, Special_Footprints:BoyKisser11x11mm, F.Cu at (129.1, 125.1)
- moved H2 156.1 mm to (185.0, 67.5)
- moved H4 133.0 mm to (184.5, 129.6)
- moved H1 99.7 mm to (110.8, 67.6)
- moved H3 63.4 mm to (110.9, 129.4)
- moved J1 20.0 mm to (119.2, 69.9)
- moved J2 20.0 mm to (116.6, 111.7)
- moved R1 20.0 mm to (145.7, 81.7)
- moved R10 20.0 mm to (181.0, 115.9)
- moved R11 20.0 mm to (181.0, 119.7)
- moved R12 20.0 mm to (181.1, 123.5)
- moved R13 20.0 mm to (174.3, 74.6)
- moved R14 20.0 mm to (168.1, 74.6)
- moved R2 20.0 mm to (145.7, 85.8)
- moved R6 20.0 mm to (155.3, 74.6)
- moved R7 20.0 mm to (145.6, 77.6)
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Other:
- board outline added: 80 x 67.8 mm
- board text added: "24 SECOND COUNTER"
- board text added: "Design Engineer: Mark Garcia Date: 13 Apr 2026"
